Commit message: Rebase from 'debian/indigo/husky_description'

File: urdf/accessories/sensor_arch.urdf.xacro (robot description, xacro)
@@ -7,18 +7,14 @@
              <visual>
                  <geometry>
-                     <mesh filename="package://husky_description/meshes/accessories/${size}_mm_sensor_arch.STL" />
+                     <mesh filename="package://husky_description/meshes/accessories/${size}_mm_sensor_arch.dae" />
                  </geometry>
-                 <material name="Grey" />
              </visual>
              <collision>
                  <origin xyz="0 0 0" rpy="0 0 0"/>
                  <geometry>
-                     <mesh filename="package://husky_description/meshes/accessories/${size}_mm_sensor_arch.STL" />
+                     <mesh filename="package://husky_description/meshes/accessories/${size}_mm_sensor_arch.dae" />
                  </geometry>
              </collision>
         </link>
-        <gazebo reference="${prefix}sensor_arch_mount_link">
-            <material>Gazebo/DarkGrey</material>
-        </gazebo>
         <!-- Attach the sensor arch to the top plate -->
         <joint name="${prefix}sensor_arch_mount" type="fixed">

File: urdf/accessories/sick_lms100.urdf.xacro (robot description, xacro)
@@ -42,7 +42,6 @@
         <origin xyz="0 0 0" rpy="0 0 0" />
         <geometry>
-          <mesh filename="package://husky_description/meshes/accessories/sick_lms100.stl" />
+          <mesh filename="package://husky_description/meshes/accessories/sick_lms100.dae" />
         </geometry>
-        <material name="DarkGrey" />
       </visual>
       <collision>

File: urdf/decorations.urdf.xacro (robot description, xacro)
@@ -28,14 +28,7 @@
         <origin xyz="0 0 0" rpy="0 0 0" />
         <geometry>
-          <mesh filename="package://husky_description/meshes/top_chassis.stl" />
+          <mesh filename="package://husky_description/meshes/top_chassis.dae" />
         </geometry>
-        <material name="Yellow" />
       </visual>
-      <collision>
-        <origin xyz="0 0 0" rpy="0 0 0"/>
-        <geometry>
-          <mesh filename="package://husky_description/meshes/top_chassis.stl" />
-        </geometry>
-      </collision>
     </link>
     <!-- Attach chassis to the robot -->
@@ -44,14 +37,10 @@
       <child link="top_chassis_link" />
     </joint>
-    <gazebo reference="top_chassis_link">
-      <material>Gazebo/Yellow</material>
-    </gazebo>
     <!-- Spawn user rails -->
     <link name="user_rail_link">
       <visual>
         <geometry>
-          <mesh filename="package://husky_description/meshes/user_rail.stl" />
+          <mesh filename="package://husky_description/meshes/user_rail.dae" />
         </geometry>
-        <material name="DarkGrey" />
       </visual>
     </link>
@@ -62,14 +51,10 @@
       <child link="user_rail_link" />
     </joint>
-    <gazebo reference="user_rail_link">
-      <material>Gazebo/DarkGrey</material>
-    </gazebo>
     <!-- Spawn front bumper link -->
     <link name="front_bumper_link">
       <visual>
         <geometry>
-          <mesh filename="package://husky_description/meshes/bumper.stl" />
+          <mesh filename="package://husky_description/meshes/bumper.dae" />
         </geometry>
-        <material name="DarkGrey" />
       </visual>
     </link>
@@ -80,14 +65,10 @@
       <child link="front_bumper_link" />
     </joint>
-    <gazebo reference="front_bumper_link">
-      <material>Gazebo/DarkGrey</material>
-    </gazebo>
     <!-- Spawn rear bumper link -->
     <link name="rear_bumper_link">
       <visual>
         <geometry>
-          <mesh filename="package://husky_description/meshes/bumper.stl" />
+          <mesh filename="package://husky_description/meshes/bumper.dae" />
         </geometry>
-        <material name="DarkGrey" />
       </visual>
     </link>
@@ -98,7 +79,4 @@
       <child link="rear_bumper_link" />
     </joint>
-    <gazebo reference="rear_bumper_link">
-      <material>Gazebo/DarkGrey</material>
-    </gazebo>
     <!-- Spawn the top plate -->
     <link name="top_plate_link">
@@ -106,12 +84,11 @@
         <origin xyz="0 0 0" rpy="0 0 0" />
         <geometry>
-          <mesh filename="package://husky_description/meshes/top_plate.stl" />
+          <mesh filename="package://husky_description/meshes/top_plate.dae" />
         </geometry>
-        <material name="Black" />
       </visual>
       <collision>
         <origin xyz="0 0 0" rpy="0 0 0"/>
         <geometry>
-          <mesh filename="package://husky_description/meshes/top_plate.stl" />
+          <mesh filename="package://husky_description/meshes/top_plate.dae" />
         </geometry>
       </collision>
@@ -123,7 +100,4 @@
       </collision>
     </link>
-    <gazebo reference="top_plate_link">
-      <material>Gazebo/DarkGrey</material>
-    </gazebo>
     <!-- Attach top plate -->
     <joint name="top_plate_joint" type="fixed">

File: urdf/husky.urdf.xacro (robot description, xacro)
@@ -24,12 +24,9 @@
   <!-- Included URDF/XACRO Files -->
   <xacro:include filename="$(find husky_description)/urdf/decorations.urdf.xacro" />
+  <xacro:include filename="$(find husky_description)/urdf/wheel.urdf.xacro" />
   <xacro:include filename="$(find husky_description)/urdf/accessories/kinect_camera.urdf.xacro"/>
   <xacro:include filename="$(find husky_description)/urdf/accessories/sick_lms100.urdf.xacro"/>
   <xacro:include filename="$(find husky_description)/urdf/accessories/sensor_arch.urdf.xacro"/>
-  <!-- <xacro:include filename="$(find robotiq_c2_model_visualization)/urdf/robotiq_c2_model_macro.xacro"/> -->
   <xacro:include filename="$(find ur_description)/urdf/ur5.urdf.xacro" />
-  <!-- Included URDF/XACRO Files -->
-  <xacro:include filename="$(find husky_description)/urdf/materials.urdf" />
-  <xacro:include filename="$(find husky_description)/urdf/wheel.urdf.xacro" />
   <property name="M_PI" value="3.14159"/>
   <!-- Base Size -->
@@ -45,22 +42,11 @@
   <xacro:property name="wheel_radius" value="0.17775" />
   <xacro:macro name="husky_robot">
-    <!-- Base link is on the ground under the robot -->
-    <link name="base_footprint"/>
-    <gazebo reference="base_footprint">
-      <material>Gazebo/DarkGrey</material>
-    </gazebo>
-    <joint name="chassis_joint" type="fixed">
-      <origin xyz="0 0 ${wheel_radius - wheel_vertical_offset}" rpy="0 0 0" />
-      <parent link="base_footprint" />
-      <child link="base_link" />
-    </joint>
-    <!-- Chassis link is the center of the robot's bottom plate -->
+    <!-- Base link is the center of the robot's bottom plate -->
     <link name="base_link">
       <visual>
         <origin xyz="0 0 0" rpy="0 0 0" />
         <geometry>
-          <mesh filename="package://husky_description/meshes/base_link.stl" />
+          <mesh filename="package://husky_description/meshes/base_link.dae" />
         </geometry>
-        <material name="Black" />
       </visual>
       <collision>
@@ -76,4 +62,14 @@
         </geometry>
       </collision>
+    </link>
+    <!-- Base footprint is on the ground under the robot -->
+    <link name="base_footprint"/>
+    <joint name="base_footprint_joint" type="fixed">
+      <origin xyz="0 0 ${wheel_vertical_offset - wheel_radius}" rpy="0 0 0" />
+      <parent link="base_link" />
+      <child link="base_footprint" />
+    </joint>
+    <!-- Interial link stores the robot's inertial information -->
+    <link name="inertial_link">
       <inertial>
         <mass value="33.455" />
@@ -82,6 +78,9 @@
       </inertial>
     </link>
-    <gazebo reference="base_link">
-    </gazebo>
+    <joint name="inertial_joint" type="fixed">
+      <origin xyz="0 0 0" rpy="0 0 0" />
+      <parent link="base_link" />
+      <child link="inertial_link" />
+    </joint>
     <!-- IMU Link is the standard mounting position for the UM6 IMU.-->
     <!-- Can be modified with environment variables in /etc/ros/setup.bash -->

File: urdf/wheel.urdf.xacro (robot description, xacro)
@@ -32,7 +32,6 @@
 				<origin xyz="0 0 0" rpy="0 0 0" />
 				<geometry>
-					<mesh filename="package://husky_description/meshes/wheel.stl" />
+					<mesh filename="package://husky_description/meshes/wheel.dae" />
 				</geometry>
-				<material name="DarkGrey" />
 			</visual>
 			<collision>
@@ -49,6 +48,4 @@
 			<kd value="1.0" />
 			<fdir1 value="1 0 0"/>
-			<material>Gazebo/Grey</material>
-			<turnGravityOff>false</turnGravityOff>
 		</gazebo>
 		<joint name="${wheel_prefix}_wheel" type="continuous">
