Commit message: Imported upstream version '0.2.4' of 'upstream'

File: husky_description/urdf/decorations.urdf.xacro (robot description, xacro)
@@ -79,31 +79,33 @@
       <child link="rear_bumper_link" />
     </joint>
-    <!-- Spawn the top plate -->
-    <link name="top_plate_link">
-      <visual>
-        <origin xyz="0 0 0" rpy="0 0 0" />
-        <geometry>
-          <mesh filename="package://husky_description/meshes/top_plate.dae" />
-        </geometry>
-      </visual>
-      <collision>
-        <origin xyz="0 0 0" rpy="0 0 0"/>
-        <geometry>
-          <mesh filename="package://husky_description/meshes/top_plate.dae" />
-        </geometry>
-      </collision>
-      <collision>
-        <!-- Extra collision tag for widgets typically attached to top plate -->
-        <geometry>
-          <box size="0.32 0.41 0.09" rpy="0 0 0"/>
-        </geometry>
-      </collision>
-    </link>
-    <!-- Attach top plate -->
-    <joint name="top_plate_joint" type="fixed">
-      <parent link="base_link" />
-      <child link="top_plate_link"/>
-      <origin xyz="0.0812 0 0.245" rpy="0 0 0"/>
-    </joint>
+    <xacro:if value="$(optenv HUSKY_TOP_PLATE_ENABLED true)">
+      <!-- Spawn the top plate -->
+      <link name="top_plate_link">
+        <visual>
+          <origin xyz="0 0 0" rpy="0 0 0" />
+          <geometry>
+            <mesh filename="package://husky_description/meshes/top_plate.dae" />
+          </geometry>
+        </visual>
+        <collision>
+          <origin xyz="0 0 0" rpy="0 0 0"/>
+          <geometry>
+            <mesh filename="package://husky_description/meshes/top_plate.dae" />
+          </geometry>
+        </collision>
+        <collision>
+          <!-- Extra collision tag for widgets on top plate -->
+          <geometry>
+            <box size="0.32 0.41 0.09" rpy="0 0 0"/>
+          </geometry>
+        </collision>
+      </link>
+      <!-- Attach top plate -->
+      <joint name="top_plate_joint" type="fixed">
+        <parent link="base_link" />
+        <child link="top_plate_link"/>
+        <origin xyz="0.0812 0 0.245" rpy="0 0 0"/>
+      </joint>
+    </xacro:if>
   </xacro:macro>
 </robot>
