Commit message: Imported upstream version '0.2.6' of 'upstream'

File: husky_description/urdf/husky.urdf.xacro (robot description, xacro)
@@ -150,5 +150,5 @@
       </xacro:sensor_arch>
       <joint name="kinect_frame_joint" type="fixed">
-        <origin xyz="$(optenv HUSKY_KINECT_XYZ 0 0 0)" rpy="$(optenv HUSKY_KINECT_RPY 0 0.3925 3.14)" />
+        <origin xyz="$(optenv HUSKY_KINECT_XYZ 0 0 0)" rpy="$(optenv HUSKY_KINECT_RPY 0 0.18 3.14)" />
         <parent link="sensor_arch_mount_link"/>
         <child link="camera_link"/>
