Commit message: Imported upstream version '0.2.5' of 'upstream'

File: husky_description/urdf/accessories/sick_lms100.urdf.xacro (robot description, xacro)
@@ -26,7 +26,7 @@
 -->
 <robot xmlns:xacro="http://ros.org/wiki/xacro" name="sick_lms100">
-  <xacro:property name="laser_x" value="0.105" />
-  <xacro:property name="laser_y" value="0.102" />
-  <xacro:property name="laser_z" value="0.152" />
+  <xacro:property name="laser_x" value="0.11" />
+  <xacro:property name="laser_y" value="0.11" />
+  <xacro:property name="laser_z" value="0.2" />
   <xacro:property name="laser_mass" value="1.1" />
   <xacro:macro name="sick_lms100" params="prefix:=base">

File: husky_description/urdf/husky.urdf.xacro (robot description, xacro)
@@ -119,7 +119,26 @@
     </xacro:if>
     <xacro:if value="$(arg laser_enabled)">
-      <joint name="base_laser_mount" type="fixed">
-        <origin xyz="-0.07 0 0.1" rpy="0 0 0" />
-        <parent link="front_bumper_link" />
+      <joint name="laser_mount_joint" type="fixed">
+        <origin xyz="$(optenv HUSKY_LMS1XX_XYZ 0.2206 0.0 0.00635)" rpy="$(optenv HUSKY_LMS1XX_RPY 0.0 0.0 0.0)" />
+        <parent link="top_plate_link" />
+        <child link="laser_mount_link" />
+      </joint>
+      <link name="laser_mount_link">
+        <visual>
+          <origin xyz="0 0 0" rpy="0 0 ${-M_PI/2}" />
+          <geometry>
+            <mesh filename="package://husky_description/meshes/accessories/lms1xx_mount.dae" />
+          </geometry>
+        </visual>
+        <collision>
+          <origin xyz="0 0 .0585" rpy="0 0 0" />
+          <geometry>
+            <box size=".1 .108 .117" />
+          </geometry>
+        </collision>
+      </link>
+      <joint name="base_laser_joint" type="fixed">
+        <origin xyz="0.0352 0 0.0566" rpy="${M_PI} 0 0" />
+        <parent link="laser_mount_link" />
         <child link="base_laser" />
       </joint>
