Commit message: Imported upstream version '0.2.7' of 'upstream'

File: husky_description/urdf/accessories/sick_lms1xx_mount.urdf.xacro (robot description, xacro)
@@ -2,5 +2,5 @@
 <!--
 Copyright (c) 2013, Goncalo Cabrita, ISR University of Coimbra
-Copyright (c) 2014, Clearpath Robotics
+Copyright (c) 2014, 2015 Clearpath Robotics
 All rights reserved.
 Redistribution and use in source and binary forms, with or without
@@ -25,31 +25,29 @@
 SOFTWARE, EVEN IF ADVISED OF THE POSSIBILITY OF SUCH DAMAGE.
 -->
-<robot xmlns:xacro="http://ros.org/wiki/xacro" name="sick_lms100">
-  <xacro:property name="laser_x" value="0.11" />
-  <xacro:property name="laser_y" value="0.11" />
-  <xacro:property name="laser_z" value="0.2" />
-  <xacro:property name="laser_mass" value="1.1" />
-  <xacro:macro name="sick_lms100" params="prefix:=base">
-    <link name="${prefix}_laser">
-      <inertial>
-        <mass value="${laser_mass}" />
-        <origin xyz="0 0 0" />
-        <inertia ixx="${0.0833333 * laser_mass * (laser_y*laser_y + laser_z*laser_z)}" ixy="0.0" ixz="0.0"
-          iyy="${0.0833333 * laser_mass * (laser_x*laser_x + laser_z*laser_z)}" iyz="0.0"
-          izz="${0.0833333 * laser_mass * (laser_x*laser_x + laser_y*laser_y)}" />
-      </inertial>
+<robot xmlns:xacro="http://ros.org/wiki/xacro">
+  <xacro:include filename="$(find lms1xx)/urdf/sick_lms1xx.urdf.xacro" />
+  <xacro:macro name="sick_lms1xx_mount" params="prefix topic">
+  <sick_lms1xx frame="${prefix}_laser" topic="${topic}" />
+    <link name="${prefix}_laser_mount">
       <visual>
-        <origin xyz="0 0 0" rpy="0 0 0" />
+        <origin xyz="0 0 0" rpy="0 0 ${-M_PI/2}" />
         <geometry>
-          <mesh filename="package://husky_description/meshes/accessories/sick_lms100.dae" />
+          <!-- Origin of this mesh is the base of the bracket. -->
+          <mesh filename="package://husky_description/meshes/accessories/lms1xx_mount.dae" />
         </geometry>
       </visual>
       <collision>
-        <origin xyz="0 0 -0.05" rpy="0 0 0" />
+        <origin xyz="0 0 .0585" rpy="0 0 0" />
         <geometry>
-          <box size="${laser_x} ${laser_y} ${laser_z}" />
+          <box size=".1 .108 .117" />
         </geometry>
       </collision>
     </link>
+    <joint name="${prefix}_laser_joint" type="fixed">
+      <!-- This offset is from the base of the bracket to the LIDAR's focal point. -->
+      <origin xyz="0.0352 0 0.0566" rpy="${M_PI} 0 0" />
+      <parent link="${prefix}_laser_mount" />
+      <child link="${prefix}_laser" />
+    </joint>
   </xacro:macro>
 </robot>

File: husky_description/urdf/husky.urdf.xacro (robot description, xacro)
@@ -26,5 +26,5 @@
   <xacro:include filename="$(find husky_description)/urdf/wheel.urdf.xacro" />
   <xacro:include filename="$(find husky_description)/urdf/accessories/kinect_camera.urdf.xacro"/>
-  <xacro:include filename="$(find husky_description)/urdf/accessories/sick_lms100.urdf.xacro"/>
+  <xacro:include filename="$(find husky_description)/urdf/accessories/sick_lms1xx_mount.urdf.xacro"/>
   <xacro:include filename="$(find husky_description)/urdf/accessories/sensor_arch.urdf.xacro"/>
   <xacro:include filename="$(find ur_description)/urdf/ur5.urdf.xacro" />
@@ -119,29 +119,11 @@
     </xacro:if>
     <xacro:if value="$(arg laser_enabled)">
+      <sick_lms1xx_mount prefix="base" topic="scan"/>
       <joint name="laser_mount_joint" type="fixed">
-        <origin xyz="$(optenv HUSKY_LMS1XX_XYZ 0.2206 0.0 0.00635)" rpy="$(optenv HUSKY_LMS1XX_RPY 0.0 0.0 0.0)" />
+        <origin xyz="$(optenv HUSKY_LMS1XX_XYZ 0.2206 0.0 0.00635)"
+                rpy="$(optenv HUSKY_LMS1XX_RPY 0.0 0.0 0.0)" />
         <parent link="top_plate_link" />
-        <child link="laser_mount_link" />
+        <child link="base_laser_mount" />
       </joint>
-      <link name="laser_mount_link">
-        <visual>
-          <origin xyz="0 0 0" rpy="0 0 ${-M_PI/2}" />
-          <geometry>
-            <mesh filename="package://husky_description/meshes/accessories/lms1xx_mount.dae" />
-          </geometry>
-        </visual>
-        <collision>
-          <origin xyz="0 0 .0585" rpy="0 0 0" />
-          <geometry>
-            <box size=".1 .108 .117" />
-          </geometry>
-        </collision>
-      </link>
-      <joint name="base_laser_joint" type="fixed">
-        <origin xyz="0.0352 0 0.0566" rpy="${M_PI} 0 0" />
-        <parent link="laser_mount_link" />
-        <child link="base_laser" />
-      </joint>
-      <xacro:sick_lms100 prefix="base" />
     </xacro:if>
     <xacro:if value="$(arg kinect_enabled)">
